File: Optitest/Optitest.kicad_pcb (KiCad board)
At the start: 2 copper layers, 41.9 x 41.6 mm, 22 parts, among them J1 Conn_MALO, J2 Conn_REGULAR, J3 Conn_BUENO, J4 Conn_EXCELENTE, J5 Programmer, J6 Battery, SW5 SW_CONF, U1 ESP-12E, U2 L78L33_SOT89

Commit message: Opitest 11FEB23
Routing:
- net GND: track 0.00 -> 124.5 mm, vias 0 -> 1
- net VCC: track 0.00 -> 103.1 mm, vias 0 -> 3
- net /BAT: track 0.00 -> 50.6 mm
- net /Buzzer_1: track 0.00 -> 49.3 mm, vias 0 -> 1
- net /INF: track 0.00 -> 41.0 mm
- net /CONF: track 0.00 -> 27.0 mm, vias 0 -> 1
- net /RXD: track 0.00 -> 26.2 mm
- net /TXD: track 0.00 -> 24.0 mm
- net /MALO: track 0.00 -> 23.9 mm
- net /To_R5: track 0.00 -> 22.2 mm
- net /EXCELENTE: track 0.00 -> 20.0 mm
- net /REGULAR: track 0.00 -> 18.2 mm
- net /BUENO: track 0.00 -> 16.9 mm
- net Net-(SW5-Pad2): track 0.00 -> 12.5 mm
- net /To_ADC_2: track 0.00 -> 9.35 mm
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Other:
- board size 41.9 x 41.6 mm -> 39.4 x 41.9 mm
- board text added: "Opitest V2 10FEB23"
- board text added: "www.dali.com.co"
