File: Optitest/Optitest.sch (KiCad schematic (older format))
At the start: 22 parts, among them J1 Conn_MALO, J2 Conn_REGULAR, J3 Conn_BUENO, J4 Conn_EXCELENTE, J5 Programmer, J6 Battery, SW5 SW_CONF, U1 ESP-12E, U2 L78L33_SOT89

Commit message: Opitest 11FEB23
Parts:
- BZ1: footprint Altera:5V_buzzer -> Header:PinHeader_2x01_P1.27mm_Horizontal
- D1: footprint Led:D_A-405_P2.54mm_Vertical_KathodeUp -> Header:PinHeader_2x01_P1.27mm_Horizontal
- J1, J2, J3, J4, J6: footprint Header:PinHeader_2x01_P1.27mm_Vertical -> Header:PinHeader_2x01_P1.27mm_Horizontal
- SW5: footprint Conf:Push_E-Switch_KS01Q01 -> Conf:SW_PUSH-12mm
Changed lines of the file:
@@
 F 0 "SW5" H 2900 5067 50  0000 C CNN
 F 1 "SW_CONF" H 2900 4976 50  0000 C CNN
-F 2 "Conf:Push_E-Switch_KS01Q01" H 2900 4700 50  0001 C CNN
+F 2 "Conf:SW_PUSH-12mm" H 2900 4700 50  0001 C CNN
 F 3 "~" H 2900 4700 50  0001 C CNN
 	1    2900 4700
@@
 F 0 "D1" V 7289 1182 50  0000 R CNN
 F 1 "LED" V 7198 1182 50  0000 R CNN
-F 2 "Led:D_A-405_P2.54mm_Vertical_KathodeUp" H 7250 1300 50  0001 C CNN
+F 2 "Header:PinHeader_2x01_P1.27mm_Horizontal" H 7250 1300 50  0001 C CNN
 F 3 "~" H 7250 1300 50  0001 C CNN
 	1    7250 1300
@@
 F 0 "BZ1" H 8152 1329 50  0000 L CNN
 F 1 "Buzzer" H 8152 1238 50  0000 L CNN
-F 2 "Altera:5V_buzzer" V 7975 1400 50  0001 C CNN
+F 2 "Header:PinHeader_2x01_P1.27mm_Horizontal" V 7975 1400 50  0001 C CNN
 F 3 "~" V 7975 1400 50  0001 C CNN
 	1    8000 1300
@@
 F 0 "J1" H 2850 1967 50  0000 C CNN
 F 1 "Conn_MALO" H 2850 1876 50  0000 C CNN
-F 2 "Header:PinHeader_2x01_P1.27mm_Vertical" H 2800 1750 50  0001 C CNN
+F 2 "Header:PinHeader_2x01_P1.27mm_Horizontal" H 2800 1750 50  0001 C CNN
 F 3 "~" H 2800 1750 50  0001 C CNN
 	1    2800 1750
@@
 F 0 "J2" H 2850 2667 50  0000 C CNN
 F 1 "Conn_REGULAR" H 2850 2576 50  0000 C CNN
-F 2 "Header:PinHeader_2x01_P1.27mm_Vertical" H 2800 2450 50  0001 C CNN
+F 2 "Header:PinHeader_2x01_P1.27mm_Horizontal" H 2800 2450 50  0001 C CNN
 F 3 "~" H 2800 2450 50  0001 C CNN
 	1    2800 2450
@@
 F 0 "J3" H 2850 3367 50  0000 C CNN
 F 1 "Conn_BUENO" H 2850 3276 50  0000 C CNN
-F 2 "Header:PinHeader_2x01_P1.27mm_Vertical" H 2800 3150 50  0001 C CNN
+F 2 "Header:PinHeader_2x01_P1.27mm_Horizontal" H 2800 3150 50  0001 C CNN
 F 3 "~" H 2800 3150 50  0001 C CNN
 	1    2800 3150
@@
 F 0 "J4" H 2850 4067 50  0000 C CNN
 F 1 "Conn_EXCELENTE" H 2850 3976 50  0000 C CNN
-F 2 "Header:PinHeader_2x01_P1.27mm_Vertical" H 2800 3850 50  0001 C CNN
+F 2 "Header:PinHeader_2x01_P1.27mm_Horizontal" H 2800 3850 50  0001 C CNN
 F 3 "~" H 2800 3850 50  0001 C CNN
 	1    2800 3850
@@
 F 0 "J6" H 8478 3176 50  0000 L CNN
 F 1 "Battery" H 8478 3085 50  0000 L CNN
-F 2 "Header:PinHeader_2x01_P1.27mm_Vertical" H 8450 3200 50  0001 C CNN
+F 2 "Header:PinHeader_2x01_P1.27mm_Horizontal" H 8450 3200 50  0001 C CNN
 F 3 "~" H 8450 3200 50  0001 C CNN
 	1    8450 3200
